File: pikas-pcbs.kicad_pcb (KiCad board)
At the start: 2 copper layers, 24 parts, among them SW1 SW_Push, U1 ATmega32U4-AU, Y1 Crystal_GND24_Small

Commit message: Forgotten check
Parts:
- C1, C2, C3, C5, C6, C7, D1, D2, D3, D4, R4, U1: moved to B.Cu
- Y1: value Crystal_GND24_Small -> 16MHz; moved to B.Cu
- moved D4 46.6 mm to (77.8, 70.5), turned to 90 degrees
- moved Y1 38.7 mm to (61.3, 16.4), turned to 180 degrees
- moved MX4 38.1 mm to (69.6, 70.2)
- moved C2 37.9 mm to (57.0, 16.7), turned to 270 degrees
- moved R4 36.6 mm to (52.9, 20.2), turned to 270 degrees
- moved MX2 34.8 mm to (69.6, 51.2)
- moved C1 34.3 mm to (65.5, 16.4), turned to 90 degrees
- moved C3 30.5 mm to (50.4, 30.0), turned to 180 degrees
- moved D1 28.0 mm to (58.7, 51.4), turned to 90 degrees
- moved C7 25.6 mm to (57.2, 39.1)
- moved D3 25.0 mm to (58.7, 70.5), turned to 90 degrees
- moved MX1 22.5 mm to (50.6, 51.3)
- moved C5 21.6 mm to (70.0, 25.8), turned to 90 degrees
- moved C4 18.8 mm to (106.5, 37.2)
- moved R1 18.8 mm to (86.3, 58.8)
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